Commit message: Add xacro for find meshes

File: urdf/mocca.urdf (robot description, URDF)
Before this commit: robot mocca, 20 links, 19 joints
Links:
- removed link link_body_rear
- removed link link_left_lower2
- removed link link_left_upper2
- removed link link_right_lower2
- removed link link_right_upper2
- link base_link: geometry visual mesh filename=file:///home/parallels/catkin_ws/src/mocca_description/mesh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 scale=0.001 0.001 0.001
- link link_body_panelF: geometry visual mesh filename=file:///home/parallels/catkin_ws/src/mocca_description/mesh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 scale=0.001 0.001 0.001
- link link_head_pitch: geometry visual mesh filename=file:///home/parallels/catkin_ws/src/mocca_description/mesh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 scale=0.001 0.001 0.001
- link link_head_plate: geometry visual mesh filename=file:///home/parallels/catkin_ws/src/mocca_description/mesh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 scale=0.001 0.001 0.001
- link link_left_fist: geometry visual mesh filename=file:///home/parallels/catkin_ws/src/mocca_description/mesh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 scale=0.001 0.001 0.001
- link link_left_lower: geometry visual mesh filename=file:///home/parallels/catkin_ws/src/mocca_description/mesh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 scale=0.001 0.001 0.001
- link link_left_shoulder: geometry visual mesh filename=file:///home/parallels/catkin_ws/src/mocca_description/mesh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 scale=0.001 0.001 0.001
- link link_left_upper: geometry visual mesh filename=file:///home/parallels/catkin_ws/src/mocca_description/mesh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 scale=0.001 0.001 0.001
- link link_neck_lower: geometry visual mesh filename=file:///home/parallels/catkin_ws/src/mocca_description/mesh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 scale=0.001 0.001 0.001
- link link_neck_upper: geometry visual mesh filename=file:///home/parallels/catkin_ws/src/mocca_description/mesh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 scale=0.001 0.001 0.001
- link link_neck_yaw: geometry visual mesh filename=file:///home/parallels/catkin_ws/src/mocca_description/mesh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 scale=0.001 0.001 0.001
- link link_right_fist: geometry visual mesh filename=file:///home/parallels/catkin_ws/src/mocca_description/mesh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 scale=0.001 0.001 0.001
- link link_right_lower: geometry visual mesh filename=file:///home/parallels/catkin_ws/src/mocca_description/mesh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 scale=0.001 0.001 0.001
- link link_right_shoulder: geometry visual mesh filename=file:///home/parallels/catkin_ws/src/mocca_description/mesh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 scale=0.001 0.001 0.001
- link link_right_upper: geometry visual mesh filename=file:///home/parallels/catkin_ws/src/mocca_description/mesh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 scale=0.001 0.001 0.001
Joints:
- removed joint joint_body_rear
- removed joint joint_left_2_extra
- removed joint joint_left_3_extra
- removed joint joint_right_2_extra
- removed joint joint_right_3_extra

Commit message: remove files that not use

File: urdf/mocca.urdf (robot description, URDF)
Before this commit: robot mocca, 15 links, 14 joints
Joints:
- removed joint joint_neck_yaw
- added joint joint_head_yaw: type revolute, parent base_link, child link_neck_yaw, origin xyz=-0.02 0 0.195 rpy=0 0 0, axis 0 0 1, limit lower=-1.57 upper=1.57 effort=1000.0 velocity=0.5
- joint joint_head_pitch: limit (none) -> lower=-1.57 upper=1.57 effort=1000.0 velocity=0.5; type continuous -> revolute
- joint joint_left_1: limit (none) -> lower=-1.57 upper=1.57 effort=1000.0 velocity=0.5; type continuous -> revolute
- joint joint_left_2: limit (none) -> lower=-1.57 upper=1.57 effort=1000.0 velocity=0.5; type continuous -> revolute
- joint joint_left_3: limit (none) -> lower=-1.57 upper=1.57 effort=1000.0 velocity=0.5; type continuous -> revolute
- joint joint_right_1: limit (none) -> lower=-1.57 upper=1.57 effort=1000.0 velocity=0.5; type continuous -> revolute
- joint joint_right_2: limit (none) -> lower=-1.57 upper=1.57 effort=1000.0 velocity=0.5; type continuous -> revolute
- joint joint_right_3: limit (none) -> lower=-1.57 upper=1.57 effort=1000.0 velocity=0.5; type continuous -> revolute

File: urdf/mocca.xacro (robot description, xacro)
@@ -3,4 +3,5 @@
   <xacro:property name="obj_scale" value="0.001 0.001 0.001" />
   <xacro:property name="pkg_path" value='$(find mocca_description)' />
+  <xacro:property name="convert_command" value='xacro --inorder mocca.xacro > mocca.urdf' />
   <material name="Brown">
     <color rgba="0.4823 0.3843 0.2666 1"/>
@@ -33,9 +34,10 @@
   </link>
   <!-- NECK START-->
-  <joint name="joint_neck_yaw" type="continuous">
+  <joint name="joint_head_yaw" type="revolute">
     <parent link="base_link"/>
     <child link="link_neck_yaw"/>
     <axis rpy="0 0 0" xyz="0 0 1"/>
     <origin rpy="0 0 0" xyz="-0.02 0 0.195"/>
+    <limit effort="1000.0" lower="-1.57" upper="1.57" velocity="0.5"/>
   </joint>
   <link name="link_neck_yaw">
@@ -76,9 +78,10 @@
     </visual>
   </link>
-  <joint name="joint_head_pitch" type="continuous">
+  <joint name="joint_head_pitch" type="revolute">
     <parent link="link_neck_upper"/>
     <child link="link_head_pitch"/>
     <axis xyz="0 1 0"/>
     <origin rpy="0 0 0" xyz="0 0 0"/>
+    <limit effort="1000.0" lower="-1.57" upper="1.57" velocity="0.5"/>
   </joint>
   <link name="link_head_pitch">
@@ -106,9 +109,10 @@
   </link>
   <!-- ARM RIGHT START-->
-  <joint name="joint_right_1" type="continuous">
+  <joint name="joint_right_1" type="revolute">
     <parent link="base_link"/>
     <child link="link_right_shoulder"/>
     <axis xyz="0 1 0"/>
     <origin xyz="0.013 -0.08 0.14"/>
+    <limit effort="1000.0" lower="-1.57" upper="1.57" velocity="0.5"/>
   </joint>
   <link name="link_right_shoulder">
@@ -121,9 +125,10 @@
     </visual>
   </link>
-  <joint name="joint_right_2" type="continuous">
+  <joint name="joint_right_2" type="revolute">
     <parent link="link_right_shoulder"/>
     <child link="link_right_upper"/>
     <axis xyz="0 0 1"/>
     <origin xyz="0 -0.03 0.0"/>
+    <limit effort="1000.0" lower="-1.57" upper="1.57" velocity="0.5"/>
   </joint>
   <link name="link_right_upper">
@@ -136,24 +141,10 @@
     </visual>
   </link>
-<!--   <joint name="joint_right_2_extra" type="fixed">
-    <parent link="link_right_upper"/>
-    <child link="link_right_upper2"/>
-    <origin xyz="0 0 0"/>
-  </joint>
-  <link name="link_right_upper2">
-    <visual>
-      <geometry>
-	<mesh filename="file://${pkg_path}/meshes/MC_ARM_Upper.stl" scale='${obj_scale}'/>
-      </geometry>
-      <origin rpy="0 3.14 0" xyz="0 0 0"/>
-      <material name="Brown"/>
-    </visual>
-  </link>
- -->
-  <joint name="joint_right_3" type="continuous">
+  <joint name="joint_right_3" type="revolute">
     <parent link="link_right_upper"/>
     <child link="link_right_lower"/>
     <axis xyz="0 0 1"/>
     <origin xyz="0 -0.06 0.0"/>
+    <limit effort="1000.0" lower="-1.57" upper="1.57" velocity="0.5"/>
   </joint>
   <link name="link_right_lower">
@@ -166,19 +157,4 @@
     </visual>
   </link>
-<!--   <joint name="joint_right_3_extra" type="fixed">
-    <parent link="link_right_lower"/>
-    <child link="link_right_lower2"/>
-    <origin xyz="0 0 0"/>
-  </joint>
-  <link name="link_right_lower2">
-    <visual>
-      <geometry>
-	<mesh filename="file://${pkg_path}/meshes/MC_ARM_Lower.stl" scale='${obj_scale}'/>
-      </geometry>
-      <origin rpy="0 3.14 0" xyz="0 0 0"/>
-      <material name="Brown"/>
-    </visual>
-  </link>
- -->
   <joint name="joint_right_fist" type="fixed">
     <parent link="link_right_lower"/>
@@ -196,9 +172,10 @@
   </link>
   <!-- ARM LEFT START-->
-  <joint name="joint_left_1" type="continuous">
+  <joint name="joint_left_1" type="revolute">
     <parent link="base_link"/>
     <child link="link_left_shoulder"/>
     <axis xyz="0 1 0"/>
     <origin xyz="0.013 0.08 0.14"/>
+    <limit effort="1000.0" lower="-1.57" upper="1.57" velocity="0.5"/>
   </joint>
   <link name="link_left_shoulder">
@@ -211,9 +188,10 @@
     </visual>
   </link>
-  <joint name="joint_left_2" type="continuous">
+  <joint name="joint_left_2" type="revolute">
     <parent link="link_left_shoulder"/>
     <child link="link_left_upper"/>
     <axis xyz="0 0 1"/>
     <origin xyz="0 0.03 0.0"/>
+    <limit effort="1000.0" lower="-1.57" upper="1.57" velocity="0.5"/>
   </joint>
   <link name="link_left_upper">
@@ -226,24 +204,10 @@
     </visual>
   </link>
-<!--   <joint name="joint_left_2_extra" type="fixed">
-    <parent link="link_left_upper"/>
-    <child link="link_left_upper2"/>
-    <origin xyz="0 0 0"/>
-  </joint>
-  <link name="link_left_upper2">
-    <visual>
-      <geometry>
-	<mesh filename="file://${pkg_path}/meshes/MC_ARM_Upper.stl" scale='${obj_scale}'/>
-      </geometry>
-      <origin rpy="0 3.14 3.14" xyz="0 0 0"/>
-      <material name="Brown"/>
-    </visual>
-  </link>
- -->
-  <joint name="joint_left_3" type="continuous">
+  <joint name="joint_left_3" type="revolute">
     <parent link="link_left_upper"/>
     <child link="link_left_lower"/>
     <axis xyz="0 0 1"/>
     <origin xyz="0 0.06 0.0"/>
+    <limit effort="1000.0" lower="-1.57" upper="1.57" velocity="0.5"/>
   </joint>
   <link name="link_left_lower">
@@ -256,19 +220,4 @@
     </visual>
   </link>
-<!--   <joint name="joint_left_3_extra" type="fixed">
-    <parent link="link_left_lower"/>
-    <child link="link_left_lower2"/>
-    <origin xyz="0 0 0"/>
-  </joint>
-  <link name="link_left_lower2">
-    <visual>
-      <geometry>
-	<mesh filename="file://${pkg_path}/meshes/MC_ARM_Lower.stl" scale='${obj_scale}'/>
-      </geometry>
-      <origin rpy="0 3.14 3.14" xyz="0 0 0"/>
-      <material name="Brown"/>
-    </visual>
-  </link>
- -->
   <joint name="joint_left_fist" type="fixed">
     <parent link="link_left_lower"/>
